File: eagle/ChocoKeys/test_module.brd (EAGLE design)
At the start: 91.4 x 94 mm, 38 parts, among them Q2 4.2A/20V/35mΩ, U1 CD4532BM, U11 SN74LVC1G18DBVR, U12 WS2812B, U13 WS2812B, U14 WS2812B, U15 L7805CV, U16 SN74LVC1G3157DBVR, U2 ATTINY402-SSNR, U3 WS2812B, U4 ATTINY1607-MFR

Commit message: 32.09.2024
update eagle
Parts:
- removed C9: 0.22uF, SparkFun-Capacitors:1206
- removed Q2: 4.2A/20V/35mΩ, SparkFun-DiscreteSemi:SOT23-3
- removed R1, R2: 220, SparkFun-Resistors:0603
- removed U11: SN74LVC1G18DBVR, SN74LVC1G18DBVR:SOT95P280X145-6N
- removed U15: L7805CV, L7805CV:TO255P1040X460X1968-3
- added IC1: ATTINY426-XUR, ATTINY426-XUR:SOP65P780X200-20N
- added U5, U6, U7: SN74LVC1G18DBVR, SN74LVC1G18DBVR:SOT95P280X145-6N
- added U8: SN74LVC1G3157DBVR, SN74LVC1G3157DBVR:SOT95P280X145-6N
- U1: value CD4532BM -> SN74LVC1G18DBVR; device CD4532BM:SOIC127P600X175-16N -> SN74LVC1G18DBVR:SOT95P280X145-6N
- moved U12 56.8 mm to (22.9, 22.9)
- moved U13 56.8 mm to (68.6, 22.9)
- moved C1 36.4 mm to (38.1, 38.1), turned to 90 degrees
- moved U2 34.0 mm to (48.3, 38.9), turned to 90 degrees
- moved C6 24.3 mm to (54.6, 43.2), turned to 90 degrees
- moved C7 24.3 mm to (54.6, 38.1), turned to 90 degrees
- moved C3 23.9 mm to (41.9, 38.1), turned to 90 degrees
- moved U1 21.7 mm to (38.1, 61.0)
- moved U16 15.3 mm to (53.3, 55.9)
- moved C4 14.8 mm to (58.4, 43.2), turned to 90 degrees
- moved C5 14.8 mm to (58.4, 38.1), turned to 90 degrees
- moved U3 14.4 mm to (22.9, 71.1), turned to 180 degrees
- moved U14 14.4 mm to (68.6, 71.1), turned to 180 degrees
- moved C2 10.2 mm to (54.6, 48.3), turned to 90 degrees
- moved U4 8.03 mm to (48.3, 48.3)
Connections:
- removed net 5V: C1.1, C2.1, C3.1, C4.1, C5.1, C6.1, C7.1, R1.2, R2.2, U1.16, U1.5, U11.5, U12.1, U13.1, U14.1, U15.3, U16.5, U2.1, U3.1, U4.4
- removed net DBG: Q2.3, U11.3, U16.1
- removed net DBG_SL: U11.1, U4.13
- removed net DISC: U4.12
- removed net DISC_EN: U4.20
- removed net ENC0: U1.9, U4.17
- removed net ENC1: U1.7, U4.18
- removed net ENC2: U1.6, U4.19
- new net BUSY: IC1.7
- new net CLK: IC1.3, U1.4
- new net DBG_CORE: IC1.16, U6.4
- new net DBG_MAIN: U5.4
- new net DBG_RGB: U16.3, U6.6
- new net DBG_SL0: U4.13, U5.1
- new net DBG_SL1: U16.6, U4.12, U6.1
- new net INT_RO: IC1.5, U8.3
- new net INT_RWM: U4.11, U8.6
- new net INT_WO: IC1.4, U8.1
- new net N$4: U1.6, U5.3
- new net N$5: U5.6, U6.3
- new net PORT_0: IC1.15
- new net PORT_1: IC1.14
- new net PORT_2: IC1.13
- new net PORT_3: IC1.12
- new net PORT_4: IC1.11
- new net PORT_5: IC1.10
- new net PORT_6: IC1.9
- new net PORT_7: IC1.8
- new net SPI_SL: U4.17, U7.1
- new net SS_CORE: IC1.2, U7.4
- new net SS_RGB: U16.1, U7.6
- new net UPDI/CLK: U1.3
- net DBG_EN: now also U1.1; no longer Q2.1, U16.6
- net GND: now also IC1.20, U1.2, U5.2, U7.2, U8.2; no longer C9.2, U1.8, U11.2, U15.2
- net INT: now also U8.4; no longer U4.11
- net MAIN_DBG: no longer U11.4
- net MISO: now also IC1.18
- net MOSI: now also IC1.17
- net RGB_DBG_SS: no longer U11.6
- net SCK: now also IC1.19
- net SCL: no longer R1.1
- net SDA: no longer R2.1
- net SS: now also U7.3; no longer U16.3
- net UPDI: no longer Q2.2
- net VCC: now also C1.1, C2.1, C3.1, C4.1, C5.1, C6.1, C7.1, IC1.1, U1.5, U12.1, U13.1, U14.1, U16.5, U2.1, U3.1, U4.4, U5.5, U6.2, U6.5, U7.5, U8.5; no longer C9.1, U1.1, U1.10, U1.11, U1.12, U1.13, U1.2, U1.3, U1.4, U15.1
