File: eagle/ChocoKeys/test_module.sch (EAGLE design)
At the start: 38 parts, among them Q2 4.2A/20V/35mΩ, U1 CD4532BM, U11 SN74LVC1G18DBVR, U12 WS2812B, U13 WS2812B, U14 WS2812B, U15 L7805CV, U16 SN74LVC1G3157DBVR, U2 ATTINY402-SSNR, U3 WS2812B, U4 ATTINY1607-MFR

Commit message: 32.09.2024
update eagle
Parts:
- removed C9: 0.22uF, SparkFun-Capacitors:2.2UF-1206-50V-10%
- removed Q2: 4.2A/20V/35mΩ, SparkFun-DiscreteSemi:MOSFET-NCH-AO3404A
- removed R1, R2: 220, SparkFun-Resistors:220OHM-0603-1/10W-1%
- removed U11: SN74LVC1G18DBVR, SN74LVC1G18DBVR:SN74LVC1G18DBVR
- removed U15: L7805CV, L7805CV:L7805CV
- added IC1: ATTINY426-XUR, ATTINY426-XUR:ATTINY426-XUR
- added U5, U6, U7: SN74LVC1G18DBVR, SN74LVC1G18DBVR:SN74LVC1G18DBVR
- added U8: SN74LVC1G3157DBVR, SN74LVC1G3157DBVR:SN74LVC1G3157DBVR
- U1: value CD4532BM -> SN74LVC1G18DBVR; device CD4532BM:CD4532BM -> SN74LVC1G18DBVR:SN74LVC1G18DBVR
Connections:
- removed net 5V: C1.1, C2.1, C3.1, C4.1, C5.1, C6.1, C7.1, R1.2, R2.2, U1.EI, U1.VDD, U11.VCC, U12.VDD, U13.VDD, U14.VDD, U15.OUTPUT, U16.VCC, U2.VDD, U3.VDD, U4.VDD
- removed net DBG: Q2.D, U11.A, U16.B2
- removed net DBG_SL: U11.S, U4.PB3
- removed net DISC: U4.PB4
- removed net DISC_EN: U4.PC3
- removed net ENC0: U1.Q0, U4.PC0
- removed net ENC1: U1.Q1, U4.PC1
- removed net ENC2: U1.Q2, U4.PC2
- new net BUSY: IC1.PB4
- new net CLK: IC1.PA5, U1.Y1
- new net DBG_CORE: IC1.PA0_(UPDI/!RESET), U6.Y1
- new net DBG_MAIN: U5.Y1
- new net DBG_RGB: U16.B1, U6.Y2
- new net DBG_SL0: U4.PB3, U5.S
- new net DBG_SL1: U16.S, U4.PB4, U6.S
- new net INT_RO: IC1.PA7, U8.B1
- new net INT_RWM: U4.PB5, U8.S
- new net INT_WO: IC1.PA6, U8.B2
- new net N$4: U1.Y2, U5.A
- new net N$5: U5.Y2, U6.A
- new net PORT_0: IC1.PC3
- new net PORT_1: IC1.PC2
- new net PORT_2: IC1.PC1
- new net PORT_3: IC1.PC0
- new net PORT_4: IC1.PB0
- new net PORT_5: IC1.PB1
- new net PORT_6: IC1.(TOSC2)_PB2
- new net PORT_7: IC1.(TOSC1)_PB3
- new net SPI_SL: U4.PC0, U7.S
- new net SS_CORE: IC1.PA4, U7.Y1
- new net SS_RGB: U16.B2, U7.Y2
- new net UPDI/CLK: U1.A
- net DBG_EN: now also U1.S; no longer Q2.G, U16.S
- net GND: now also IC1.GND, U1.GND, U5.GND, U7.GND, U8.GND; no longer C9.2, U1.VSS, U11.GND, U15.GROUND
- net INT: now also U8.A; no longer U4.PB5
- net MAIN_DBG: no longer U11.Y1
- net MISO: now also IC1.PA2
- net MOSI: now also IC1.PA1
- net RGB_DBG_SS: no longer U11.Y2
- net SCK: now also IC1.PA3(EXTCLK)
- net SCL: no longer R1.1
- net SDA: no longer R2.1
- net SS: now also U7.A; no longer U16.B1
- net UPDI: no longer Q2.S
- net VCC: now also C1.1, C2.1, C3.1, C4.1, C5.1, C6.1, C7.1, IC1.VDD, U1.VCC, U12.VDD, U13.VDD, U14.VDD, U16.VCC, U2.VDD, U3.VDD, U4.VDD, U5.VCC, U6.GND, U6.VCC, U7.VCC, U8.VCC; no longer C9.1, U1.D0, U1.D1, U1.D2, U1.D3, U1.D4, U1.D5, U1.D6, U1.D7, U15.INPUT
Other:
- note added: "(BI-DIRECTIONAL)"
- note added: "ATTINY426"
- note added: "DBG SELECTION"
- note added: "INT SELECTION"
- note added: "PORTS"
- note added: "RGB SELECTION"
- note added: "UPDI SELECTION"
- note added: "mTC"
- note removed: "DBG DEMUX"
- note removed: "DBG MUX"
- note removed: "DEBUG SW"
- note removed: "ENCODER"
- note removed: "I2C BUS"
- note removed: "MTC"
- note removed: "VREG"
- moved on the sheet: C1, C2, C3, U16, U2, U4
